File: HARDWARE/NeuroBytes_Battery_Pack.sch (KiCad schematic (older format))
At the start: 16 parts, among them P1 JST_GH_5-pos, P2 JST_GH_5-pos, SW1 Switch_SPDT, U1 LDL212_LDO

Commit message: updated footprints to include outlines. re-generated Gerbers. added placement pdf.
Parts:
- C1, C2: footprint KiCad_Footprints:ZF_SMD_NonPol_0603 -> Capacitors_SMD:C_0603_HandSoldering
Changed lines of the file:
@@
 F 0 "C1" H 3625 2750 50  0000 L CNN
 F 1 "1u" H 3625 2550 50  0000 L CNN
-F 2 "KiCad_Footprints:ZF_SMD_NonPol_0603" H 3638 2500 50  0001 C CNN
+F 2 "Capacitors_SMD:C_0603_HandSoldering" H 3638 2500 50  0001 C CNN
 F 3 "" H 3600 2650 50  0000 C CNN
 F 4 "Taiyo Yuden" H 3600 2650 60  0001 C CNN "Mfr"
@@
 F 0 "C2" H 7025 2750 50  0000 L CNN
 F 1 "1u" H 7025 2550 50  0000 L CNN
-F 2 "KiCad_Footprints:ZF_SMD_NonPol_0603" H 7038 2500 50  0001 C CNN
+F 2 "Capacitors_SMD:C_0603_HandSoldering" H 7038 2500 50  0001 C CNN
 F 3 "" H 7000 2650 50  0000 C CNN
 F 4 "Taiyo Yuden" H 7000 2650 60  0001 C CNN "Mfr"
